Commit message: feat: Add autonomous navigation launch files and point cloud converter
- Created `bringup_tb3_mid360_copy.launch` and `bringup_tb3_mid360_toolbox.launch` for launching the TurtleBot3 with Mid360 sensor in a simulated environment.
- Added RViz configuration file `nav_mapping.rviz` for visualizing the robot's mapping process.
- Implemented `pointcloud_converter.py` script to convert `sensor_msgs/PointCloud` to `sensor_msgs/PointCloud2` format, facilitating compatibility with SLAM and RViz.
- Introduced a new note file `mynote` for quick reference on starting the robot control.

File: src/autonomous_navigation/urdf/turtlebot3_burger.urdf.xacro (robot description, xacro)
@@ -130,6 +130,6 @@
     <parent link="base_link"/>
     <child link="laser_livox"/>
-    <!-- Position: front-upper of chassis, Pitch 45° downward same as A1 -->
-    <origin xyz="0.04 0 0.16" rpy="0 0.785 0"/>
+    <!-- Position: front-upper of chassis, Pitch ~5° 确保最低射线接近水平可打墙 -->
+    <origin xyz="0.04 0 0.16" rpy="0 0.087 0"/>
   </joint>
   <!-- LiDAR internal IMU link (mounted inside Mid360) -->
@@ -211,5 +211,5 @@
       <wheelSeparation>0.160</wheelSeparation>
       <wheelDiameter>0.066</wheelDiameter>
-      <wheelAcceleration>1</wheelAcceleration>
+      <wheelAcceleration>10</wheelAcceleration>
       <wheelTorque>20</wheelTorque>
       <rosDebugLevel>na</rosDebugLevel>

Commit message: update

File: src/autonomous_navigation/urdf/turtlebot3_burger.urdf.xacro (robot description, xacro)
@@ -130,6 +130,6 @@
     <parent link="base_link"/>
     <child link="laser_livox"/>
-    <!-- Position: front-upper of chassis, Pitch ~5° 确保最低射线接近水平可打墙 -->
-    <origin xyz="0.04 0 0.16" rpy="0 0.087 0"/>
+    <!-- Position: front-upper of chassis, 0° pitch（水平安装，避免 IMU 重力倾斜） -->
+    <origin xyz="0.04 0 0.16" rpy="0 0 0"/>
   </joint>
   <!-- LiDAR internal IMU link (mounted inside Mid360) -->

Commit message: ``` refactor(fastlio): 更新FAST_LIO子模块状态
- FAST_LIO子模块标记为dirty状态
- LiDAR_IMU_Init子模块标记为dirty状态

docs(config): 改进Mid360外参配置文档说明

- 更新tb3_mid360_fastlio.yaml中外参注释说明
- 明确说明LiDAR→IMU外参计算方式和内部硬件偏移
- 添加关于Mid-360内部轴向对齐的注释说明

fix(launch): 修正TurtleBot3 Mid360启动文件参数

- 更新laser_livox_level坐标系的Z轴高度从0.16到0.4米
- 修改注释说明Mid360前倾45°安装方式
- 添加关于target_frame修改的使用说明

feat(mapping): 优化Fast-LIO建图参数配置

- 将filter_size_map从0.2调整到0.3以平衡精度和性能
- 更新TF变换配置以正确处理IMU倾斜补偿
- 添加Fast-LIO相机初始化水平对齐的注释说明

refactor(maps): 改进点云转2D地图算法实现

- 更新Fast-LIO初始旋转估计相关注释
- 调整地面和障碍物Z轴高度阈值参数
- 添加机器人周围强制空闲半径参数
- 重构OccupancyGrid元数据设置方式

perf(lidar): 优化点云转自定义消息时间戳处理

- 将SCAN_PERIOD_US改为SCAN_PERIOD_NS，使用纳秒单位
- 修正时间戳基准计算，减去扫描周期获得帧首时刻
- 提高时间同步精度以适配Livox协议

fix(urdf): 修正TurtleBot3 LiDAR安装角度配置

- 将laser_livox关节的俯仰角从0改为0.7854弧度（45度）
- 更新注释说明后仰45°安装的优势和Fast-LIO重力对齐功能
```

File: src/autonomous_navigation/urdf/turtlebot3_burger.urdf.xacro (robot description, xacro)
@@ -130,6 +130,6 @@
     <parent link="base_link"/>
     <child link="laser_livox"/>
-    <!-- Position: front-upper of chassis, 0° pitch（水平安装，避免 IMU 重力倾斜） -->
-    <origin xyz="0.04 0 0.16" rpy="0 0 0"/>
+    <!-- 后仰45°安装: 扩大天花板覆盖 + 后方墙壁扫描; Fast-LIO IMU 重力估计自动对齐地图 -->
+    <origin xyz="0.04 0 0.4" rpy="0 0.7854 0"/>
   </joint>
   <!-- LiDAR internal IMU link (mounted inside Mid360) -->

Commit message: ``` feat(autonomous_navigation): 添加自动导航功能包并配置Livox Mid360雷达参数
添加了完整的自主导航功能包，包括SLAM建图、路径规划和探索功能，
同时调整了Livox Mid360雷达的安装高度参数以优化环境感知效果。

- 在command.txt中添加了新的启动命令序列，包括环境配置和导航启动脚本
- 配置CMakeLists.txt以安装Python脚本和资源目录（launch/config/rviz）
- 更新URDF文件中LiDAR传感器的高度参数，从0.16m调整到0.4m
- 修改launch文件中的坐标变换和点云处理参数以适应新的传感器高度
- 移除重复的launch文件并更新依赖包列表
```

File: src/autonomous_navigation/urdf/turtlebot3_burger.urdf.xacro (robot description, xacro)
@@ -131,5 +131,5 @@
     <child link="laser_livox"/>
     <!-- Position: front-upper of chassis, Pitch ~5° 确保最低射线接近水平可打墙 -->
-    <origin xyz="0.04 0 0.16" rpy="0 0.087 0"/>
+    <origin xyz="0.04 0 0.4" rpy="0 0.087 0"/>
   </joint>
   <!-- LiDAR internal IMU link (mounted inside Mid360) -->

Commit message: update

File: src/autonomous_navigation/urdf/turtlebot3_burger.urdf.xacro (robot description, xacro)
@@ -131,5 +131,5 @@
     <child link="laser_livox"/>
     <!-- Position: front-upper of chassis, Pitch ~5° 确保最低射线接近水平可打墙 -->
-    <origin xyz="0.04 0 0.4" rpy="0 0.087 0"/>
+    <origin xyz="0.04 0 0.4" rpy="0 0.785 0"/>
   </joint>
   <!-- LiDAR internal IMU link (mounted inside Mid360) -->
