Commit message: feat: 改为gazebo标准雷达插件，并对launch文件进行适配
- 在映射发射文件中删除了点云到激光扫描的转换，直接使用 Gazebo 的 LaserScan。
- 在 Gazebo 发射文件中延迟机器人生成和控制器生成器初始化，以避免超时。从自定义 livox_laser_simulation 切换到标准 Gazebo 激光插件，以减少 CPU 负载并防止分段故障。
- 将雷达改为水平
- 下一步将修改movebase参数

File: src/unitree_guide/unitree_ros/robots/a1_description/xacro/gazebo.xacro (robot description, xacro)
@@ -278,23 +278,17 @@
     <xacro:if value="${'$(arg ENABLE_LIVOX)' == 'true'}">
         <gazebo reference="laser_livox">
-            <sensor type="ray" name="laser_livox">
+            <sensor name="laser_livox" type="ray">
+                <pose>0 0 0 0 0 0</pose>
                 <always_on>true</always_on>
-                <pose>0 0 0 0 0 0</pose>
-                <visualize>true</visualize>
                 <update_rate>10</update_rate>
+                <visualize>false</visualize>
                 <ray>
                     <scan>
                         <horizontal>
-                            <samples>100</samples>
+                            <samples>640</samples>
                             <resolution>1</resolution>
-                            <min_angle>${0}</min_angle>
-                            <max_angle>${2*M_PI}</max_angle>
+                            <min_angle>${-M_PI}</min_angle>
+                            <max_angle>${M_PI}</max_angle>
                         </horizontal>
-                        <vertical>
-                            <samples>360</samples>
-                            <resolution>1</resolution>
-                            <min_angle>${-5.22/180*M_PI}</min_angle>
-                            <max_angle>${57.22/180*M_PI}</max_angle>
-                        </vertical>
                     </scan>
                     <range>
@@ -309,36 +303,11 @@
                     </noise>
                 </ray>
-                <plugin name="gazebo_ros_laser_controller" filename="liblivox_laser_simulation.so">
-                    <ray>
-                        <scan>
-                            <horizontal>
-                                <samples>100</samples>
-                                <resolution>1</resolution>
-                                <min_angle>${0}</min_angle>
-                                <max_angle>${2*M_PI}</max_angle>
-                            </horizontal>
-                            <vertical>
-                                <samples>360</samples>
-                                <resolution>1</resolution>
-                                <min_angle>${-5.22/180*M_PI}</min_angle>
-                                <max_angle>${57.22/180*M_PI}</max_angle>
-                            </vertical>
-                        </scan>
-                        <range>
-                            <min>0.1</min>
-                            <max>40</max>
-                            <resolution>0.01</resolution>
-                        </range>
-                        <noise>
-                            <type>gaussian</type>
-                            <mean>0.0</mean>
-                            <stddev>0.005</stddev>
-                        </noise>
-                    </ray>
-                    <visualize>true</visualize>
-                    <samples>24000</samples>
-                    <downsample>1</downsample>
-                    <csv_file_name>package://a1_description/scan_mode/mid360.csv</csv_file_name>
-                    <ros_topic>/scan</ros_topic>
+                <!-- Use standard Gazebo laser plugin instead of the custom
+                     livox_laser_simulation which causes probabilistic segfaults
+                     and heavy CPU load from 24000 ODE ray collisions. -->
+                <plugin name="gazebo_ros_laser_controller"
+                        filename="libgazebo_ros_laser.so">
+                    <robotNamespace></robotNamespace>
+                    <topicName>/scan</topicName>
                     <frameName>laser_livox</frameName>
                 </plugin>

File: src/unitree_guide/unitree_ros/robots/a1_description/xacro/robot.xacro (robot description, xacro)
@@ -134,5 +134,5 @@
     </link>
     <joint name="laser_livox_joint" type="fixed">
-            <origin xyz="0.2 0 0.08" rpy="0 0.785 0"/>
+            <origin xyz="0.2 0 0.08" rpy="0 0 0"/>
             <parent link="base"/>
             <child link="laser_livox"/>
